File: Circuit_nano/Circuit_nano.kicad_sch (KiCad schematic)
At the start: 11 parts, among them J1 Encoder, J2 LCD, J3 Power, J4 Leds, J5 Temp Sensor, U1 Nano

Commit message: updating circuits
Parts:
- removed J1: Encoder, Connector_PinSocket_2.54mm:PinSocket_1x05_P2.54mm_Vertical, symbol Connector:Conn_01x05_Male
- removed J2: LCD, Connector_PinHeader_2.54mm:PinHeader_1x04_P2.54mm_Vertical, symbol Connector:Conn_01x04_Male
- removed J3: Power, Connector_TE-Connectivity:TE_826576-2_1x02_P3.96mm_Vertical, symbol Connector:Conn_01x02_Male
- removed J4: Leds, Connector_PinHeader_2.54mm:PinHeader_1x02_P2.54mm_Vertical, symbol Connector:Conn_01x02_Male
- removed J5: Temp Sensor, Connector_PinHeader_2.54mm:PinHeader_1x02_P2.54mm_Vertical, symbol Connector:Conn_01x02_Male
- added D3: DIODE, symbol pspice:DIODE
- added Encoder1: Conn_01x05_Male, Connector_PinHeader_2.54mm:PinHeader_1x05_P2.54mm_Vertical, symbol Connector:Conn_01x05_Male
- added Heater_+1, Heater_-1, Leds1: Conn_01x03_Male, Connector_PinHeader_2.54mm:PinHeader_1x03_P2.54mm_Vertical, symbol Connector:Conn_01x03_Male
- added LCD1: Conn_01x04_Male, Connector_PinHeader_2.54mm:PinHeader_1x04_P2.54mm_Vertical, symbol Connector:Conn_01x04_Male
- added PWR1, PWR_IN1: Conn_01x02_Male, Connector_PinHeader_2.54mm:PinHeader_1x02_P2.54mm_Vertical, symbol Connector:Conn_01x02_Male
- added Q1: Q_NPN_Darlington_BCE, symbol Device:Q_NPN_Darlington_BCE
- added R1: R, Resistor_SMD:R_0805_2012Metric_Pad1.20x1.40mm_HandSolder, symbol Device:R
- added Sensor1: Conn_01x02_Male, symbol Connector:Conn_01x02_Male
- renumbered R3 to R2, R2 to R3, R1 to R4
Connections:
- net +5V: now also Encoder1.1 (Pin_1), LCD1.1 (Pin_1), Sensor1.2 (Pin_2)
- net GND: now also D3.1 (K), Encoder1.2 (Pin_2), Heater_-1.1 (Pin_1), Heater_-1.2 (Pin_2), Heater_-1.3 (Pin_3), LCD1.2 (Pin_2), Leds1.1 (Pin_1), PWR1.2 (Pin_2), PWR_IN1.2 (Pin_2), Q1.3 (E)
- net at U1.23 (A4): now also LCD1.3 (Pin_3)
- net at U1.24 (A5): now also LCD1.4 (Pin_4)
- net at R2.2: now also Sensor1.1 (Pin_1)
- net at U1.7 (D4): now also Encoder1.3 (Pin_3)
- net at U1.8 (D5): now also Encoder1.4 (Pin_4)
- net at U1.9 (D6): now also Encoder1.5 (Pin_5)
- net at U1.30 (VIN): now also PWR_IN1.1 (Pin_1)
- net at R3.1: now also Leds1.2 (Pin_2)
- net at R4.1: now also Leds1.3 (Pin_3)
- net at U1.19 (A0): now also R1.1
- new net: Q1.1 (B), R1.2
- new net: D3.2 (A), Heater_+1.1 (Pin_1), Heater_+1.2 (Pin_2), Heater_+1.3 (Pin_3), PWR1.1 (Pin_1), Q1.2 (C)
- no-connect marks 21 -> 20
Other:
- moved on the sheet: D1, D2, R2, R3, R4, U1
