File: Temperature Controller Board/Temperature Controller Board.kicad_sch (KiCad schematic)
At the start: 18 parts, among them J2 Pwr, J4 AC Line, J5 Rotary Encoder Board, J6 LEDS, K1 G3MB-202PDC5 Relay, U1 AZ1117-5.0

Commit message: updated Schematic and PCB
Parts:
- removed J4: AC Line, TerminalBlock:TerminalBlock_bornier-2_P5.08mm, symbol Connector_Generic:Conn_01x02
- removed J5: Rotary Encoder Board, Connector_JST:JST_XH_B5B-XH-A_1x05_P2.50mm_Vertical, symbol 000_Thomas_Symbols:Rotary_Encoder_Board
- removed J6: LEDS, Connector_JST:JST_XH_B3B-XH-A_1x03_P2.50mm_Vertical, symbol Connector_Generic:Conn_01x03
- removed K1: G3MB-202PDC5 Relay, 000_Thomas_Footprints:G3MB-202PDC5 Relay, symbol 000_Thomas_Symbols:G3MB-202PDC5 Relay
- added J1, PWR1: Conn_01x02, Connector_JST:JST_XH_B2B-XH-A_1x02_P2.50mm_Vertical, symbol Connector_Generic:Conn_01x02
- added J4: Conn_01x05, Connector_JST:JST_XH_B5B-XH-A_1x05_P2.50mm_Vertical, symbol Connector_Generic:Conn_01x05
- added J5: Conn_01x02, 000_Thomas_Footprints:myTerminalBlock-2_P5.08mm, symbol Connector_Generic:Conn_01x02
- added K1: AQG22105, 000_Thomas_Footprints:RELAY_AQG22105, symbol 000_Thomas_Symbols:AQG22105
- A1: footprint Module:Arduino_Nano -> 000_Thomas_Footprints:Arduino Riser
- J2: value Pwr -> Conn_01x02
- LM19: renamed from LM1; footprint Connector_JST:JST_XH_B3B-XH-A_1x03_P2.50mm_Vertical -> Connector_JST:JST_XH_B3B-XH-AM_1x03_P2.50mm_Vertical
- OLED1: value ~ -> Conn_01x04
- RST1: value RST Button -> Conn_01x02; footprint Connector_PinHeader_2.54mm:PinHeader_1x02_P2.54mm_Vertical -> Connector_JST:JST_XH_B2B-XH-A_1x02_P2.50mm_Vertical
- renumbered R2 to R1, R1 to R2
Connections:
- net 5V: now also J4.2 (Pin_2)
- net CLK_en: now also J4.5 (Pin_5)
- net DT_en: now also J4.4 (Pin_4)
- net GND: now also J1.2 (Pin_2), J4.1 (Pin_1), K1.4 (IN-), PWR1.2 (Pin_2)
- net GREEN_LED: now also J2.1 (Pin_1)
- net GREEN_PIN: now also A1.6 (D3); no longer A1.2 (D0/RX)
- net RED_LED: now also J1.1 (Pin_1)
- net RED_PIN: now also A1.5 (D2); no longer A1.1 (D1/TX)
- net SWT_en: now also J4.3 (Pin_3)
- net Vin: now also PWR1.1 (Pin_1); no longer J2.1 (Pin_1)
- net relay: now also A1.12 (D9), K1.3 (IN+); no longer A1.8 (D5)
- net Aref renamed Vref
- new net: J5.1 (Pin_1), K1.2 (OUT2)
- new net: J5.2 (Pin_2), K1.1 (OUT1)
Other:
- note added: "5V Regulator for aux power"
- note added: "AC Line"
- note removed: "5V Regulator"
- moved on the sheet: C2, C3, OLED1, R1, R2, U1
